File: plug-ins/control/RedPitaya-Support/McBSP-Link-Hardware/MK3-RP-Link/rp-schield.sch (EAGLE design)
At the start: 18 parts, among them U1 SN65MLVD202A, U2 SN65MLVD202A, U3 SN65MLVD202A

Commit message: updated gnd routing
Connections:
- net GND: now also J1.3, J1.4, J1.5, J1.6
Changed lines of the file:
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@@
 <junction x="-78.74" y="144.78"/>
 <wire x1="-60.96" y1="144.78" x2="-60.96" y2="121.92" width="0.1524" layer="91"/>
+<pinref part="J1" gate="G$1" pin="3"/>
+<pinref part="J1" gate="G$1" pin="4"/>
+<wire x1="111.76" y1="121.92" x2="111.76" y2="119.38" width="0.1524" layer="91"/>
+<pinref part="J1" gate="G$1" pin="5"/>
+<wire x1="111.76" y1="119.38" x2="111.76" y2="116.84" width="0.1524" layer="91"/>
+<pinref part="J1" gate="G$1" pin="6"/>
+<wire x1="111.76" y1="114.3" x2="111.76" y2="116.84" width="0.1524" layer="91"/>
+<wire x1="111.76" y1="116.84" x2="101.6" y2="116.84" width="0.1524" layer="91"/>
+<wire x1="101.6" y1="116.84" x2="101.6" y2="175.26" width="0.1524" layer="91"/>
+<wire x1="101.6" y1="175.26" x2="104.14" y2="175.26" width="0.1524" layer="91"/>
+<wire x1="101.6" y1="175.26" x2="-7.62" y2="175.26" width="0.1524" layer="91"/>
+<wire x1="-7.62" y1="175.26" x2="-7.62" y2="170.18" width="0.1524" layer="91"/>
 </segment>
 </net>
