File: plug-ins/control/RedPitaya-Support/McBSP-Link-Hardware/MK3-RP-Link/mk3-schield-samtec-vias.sch (EAGLE design)
At the start: 13 parts, among them J4/6 ESQ-122-13-L-T, U1 SN65MLVD202A, U2 SN65MLVD202A, U3 SN65MLVD202A

Commit message: updated McBSP Link board/schematics updated FPGA bit file for (latest build for V2 Hardware/Interface), design cleanups
Parts:
- added R1, R2, R4: 100R, resistor:R-US_R0402
Connections:
- net N$1: now also R4.2
- net N$10: now also R2.1
- net N$2: now also R4.1
- net N$5: now also R1.2
- net N$6: now also R1.1
- net N$9: now also R2.2
Changed lines of the file:
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@@
 <part name="JP1" library="jumper" library_urn="urn:adsk.eagle:library:252" deviceset="JP3Q" device="" package3d_urn="urn:adsk.eagle:package:15460/1"/>
 <part name="J4/6" library="ESQ-122-13-L-T" deviceset="ESQ-122-13-L-T" device=""/>
+<part name="R4" library="resistor" library_urn="urn:adsk.eagle:library:348" deviceset="R-US_" device="R0402" package3d_urn="urn:adsk.eagle:package:26058/1" value="100R"/>
+<part name="R1" library="resistor" library_urn="urn:adsk.eagle:library:348" deviceset="R-US_" device="R0402" package3d_urn="urn:adsk.eagle:package:26058/1" value="100R"/>
+<part name="R2" library="resistor" library_urn="urn:adsk.eagle:library:348" deviceset="R-US_" device="R0402" package3d_urn="urn:adsk.eagle:package:26058/1" value="100R"/>
 </parts>
 <sheets>
@@
 </instance>
 <instance part="J4/6" gate="G$2" x="-116.84" y="96.52" rot="MR0"/>
+<instance part="R4" gate="G$1" x="60.96" y="111.76" smashed="yes" rot="R90">
+<attribute name="NAME" x="59.4614" y="107.95" size="1.778" layer="95" rot="R90"/>
+<attribute name="VALUE" x="64.262" y="107.95" size="1.778" layer="96" rot="R90"/>
+</instance>
+<instance part="R1" gate="G$1" x="60.96" y="58.42" smashed="yes" rot="R90">
+<attribute name="NAME" x="59.4614" y="54.61" size="1.778" layer="95" rot="R90"/>
+<attribute name="VALUE" x="64.262" y="54.61" size="1.778" layer="96" rot="R90"/>
+</instance>
+<instance part="R2" gate="G$1" x="60.96" y="5.08" smashed="yes" rot="R90">
+<attribute name="NAME" x="59.4614" y="1.27" size="1.778" layer="95" rot="R90"/>
+<attribute name="VALUE" x="64.262" y="1.27" size="1.778" layer="96" rot="R90"/>
+</instance>
 </instances>
 <busses>
@@
 <wire x1="88.9" y1="127" x2="88.9" y2="116.84" width="0.1524" layer="91"/>
 <pinref part="U3" gate="A" pin="A"/>
-<wire x1="88.9" y1="116.84" x2="53.34" y2="116.84" width="0.1524" layer="91"/>
+<wire x1="88.9" y1="116.84" x2="60.96" y2="116.84" width="0.1524" layer="91"/>
+<pinref part="R4" gate="G$1" pin="2"/>
+<wire x1="60.96" y1="116.84" x2="53.34" y2="116.84" width="0.1524" layer="91"/>
+<junction x="60.96" y="116.84"/>
 </segment>
 </net>
@@
 <wire x1="111.76" y1="124.46" x2="91.44" y2="124.46" width="0.1524" layer="91"/>
 <pinref part="U3" gate="A" pin="B"/>
-<wire x1="91.44" y1="124.46" x2="91.44" y2="114.3" width="0.1524" layer="91"/>
-<wire x1="91.44" y1="114.3" x2="53.34" y2="114.3" width="0.1524" layer="91"/>
+<wire x1="91.44" y1="124.46" x2="91.44" y2="106.68" width="0.1524" layer="91"/>
+<wire x1="91.44" y1="106.68" x2="60.96" y2="106.68" width="0.1524" layer="91"/>
+<wire x1="60.96" y1="106.68" x2="53.34" y2="106.68" width="0.1524" layer="91"/>
+<wire x1="53.34" y1="106.68" x2="53.34" y2="114.3" width="0.1524" layer="91"/>
+<pinref part="R4" gate="G$1" pin="1"/>
+<junction x="60.96" y="106.68"/>
 </segment>
 </net>
@@
 <wire x1="73.66" y1="73.66" x2="73.66" y2="63.5" width="0.1524" layer="91"/>
 <pinref part="U1" gate="A" pin="A"/>
-<wire x1="73.66" y1="63.5" x2="53.34" y2="63.5" width="0.1524" layer="91"/>
+<wire x1="73.66" y1="63.5" x2="60.96" y2="63.5" width="0.1524" layer="91"/>
+<pinref part="R1" gate="G$1" pin="2"/>
+<wire x1="60.96" y1="63.5" x2="53.34" y2="63.5" width="0.1524" layer="91"/>
+<junction x="60.96" y="63.5"/>
 </segment>
 </net>
@@
 <wire x1="111.76" y1="71.12" x2="76.2" y2="71.12" width="0.1524" layer="91"/>
 <pinref part="U1" gate="A" pin="B"/>
-<wire x1="76.2" y1="71.12" x2="76.2" y2="60.96" width="0.1524" layer="91"/>
-<wire x1="76.2" y1="60.96" x2="53.34" y2="60.96" width="0.1524" layer="91"/>
+<wire x1="76.2" y1="71.12" x2="76.2" y2="53.34" width="0.1524" layer="91"/>
+<wire x1="76.2" y1="53.34" x2="60.96" y2="53.34" width="0.1524" layer="91"/>
+<wire x1="60.96" y1="53.34" x2="53.34" y2="53.34" width="0.1524" layer="91"/>
+<wire x1="53.34" y1="53.34" x2="53.34" y2="60.96" width="0.1524" layer="91"/>
+<pinref part="R1" gate="G$1" pin="1"/>
+<junction x="60.96" y="53.34"/>
 </segment>
 </net>
@@
 <wire x1="93.98" y1="66.04" x2="93.98" y2="10.16" width="0.1524" layer="91"/>
 <pinref part="U2" gate="A" pin="A"/>
-<wire x1="93.98" y1="10.16" x2="53.34" y2="10.16" width="0.1524" layer="91"/>
+<wire x1="93.98" y1="10.16" x2="60.96" y2="10.16" width="0.1524" layer="91"/>
+<pinref part="R2" gate="G$1" pin="2"/>
+<wire x1="60.96" y1="10.16" x2="53.34" y2="10.16" width="0.1524" layer="91"/>
+<junction x="60.96" y="10.16"/>
 </segment>
 </net>
@@
 <segment>
 <pinref part="U2" gate="A" pin="B"/>
-<wire x1="53.34" y1="7.62" x2="96.52" y2="7.62" width="0.1524" layer="91"/>
-<wire x1="96.52" y1="7.62" x2="96.52" y2="63.5" width="0.1524" layer="91"/>
+<wire x1="53.34" y1="7.62" x2="53.34" y2="0" width="0.1524" layer="91"/>
+<wire x1="53.34" y1="0" x2="60.96" y2="0" width="0.1524" layer="91"/>
+<wire x1="60.96" y1="0" x2="96.52" y2="0" width="0.1524" layer="91"/>
+<wire x1="96.52" y1="0" x2="96.52" y2="63.5" width="0.1524" layer="91"/>
 <pinref part="J2" gate="G$1" pin="5"/>
 <wire x1="96.52" y1="63.5" x2="111.76" y2="63.5" width="0.1524" layer="91"/>
-</segment>
-</net>
+<pinref part="R2" gate="G$1" pin="1"/>
+<junction x="60.96" y="0"/>
+</segment>
+</net>

Commit message: minor updates, cleanups
Other:
- moved on the sheet: J4/6G$1, J4/6G$2

Commit message: updated FPGA init procedure updated -- next gen layout
Parts:
- added R3, R5, R6, R7, R8, R9: 25R, resistor:R-US_R0402
Connections:
- new net N$13: R3.2, U3.Y
- new net N$14: R5.2, U3.Z
- new net N$15: R6.2, U1.Y
- new net N$16: R7.2, U1.Z
- new net N$17: R8.2, U2.Y
- new net N$18: R9.2, U2.Z
- net N$11: now also R8.1; no longer U2.Y
- net N$12: now also R9.1; no longer U2.Z
- net N$3: now also R3.1; no longer U3.Y
- net N$4: now also R5.1; no longer U3.Z
- net N$7: now also R6.1; no longer U1.Y
- net N$8: now also R7.1; no longer U1.Z
Changed lines of the file:
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@@
 <part name="R1" library="resistor" library_urn="urn:adsk.eagle:library:348" deviceset="R-US_" device="R0402" package3d_urn="urn:adsk.eagle:package:26058/1" value="100R"/>
 <part name="R2" library="resistor" library_urn="urn:adsk.eagle:library:348" deviceset="R-US_" device="R0402" package3d_urn="urn:adsk.eagle:package:26058/1" value="100R"/>
+<part name="R3" library="resistor" library_urn="urn:adsk.eagle:library:348" deviceset="R-US_" device="R0402" package3d_urn="urn:adsk.eagle:package:26058/1" value="25R"/>
+<part name="R5" library="resistor" library_urn="urn:adsk.eagle:library:348" deviceset="R-US_" device="R0402" package3d_urn="urn:adsk.eagle:package:26058/1" value="25R"/>
+<part name="R6" library="resistor" library_urn="urn:adsk.eagle:library:348" deviceset="R-US_" device="R0402" package3d_urn="urn:adsk.eagle:package:26058/1" value="25R"/>
+<part name="R7" library="resistor" library_urn="urn:adsk.eagle:library:348" deviceset="R-US_" device="R0402" package3d_urn="urn:adsk.eagle:package:26058/1" value="25R"/>
+<part name="R8" library="resistor" library_urn="urn:adsk.eagle:library:348" deviceset="R-US_" device="R0402" package3d_urn="urn:adsk.eagle:package:26058/1" value="25R"/>
+<part name="R9" library="resistor" library_urn="urn:adsk.eagle:library:348" deviceset="R-US_" device="R0402" package3d_urn="urn:adsk.eagle:package:26058/1" value="25R"/>
 </parts>
 <sheets>
@@
 <attribute name="NAME" x="59.4614" y="1.27" size="1.778" layer="95" rot="R90"/>
 <attribute name="VALUE" x="64.262" y="1.27" size="1.778" layer="96" rot="R90"/>
+</instance>
+<instance part="R3" gate="G$1" x="76.2" y="127" smashed="yes" rot="R180">
+<attribute name="NAME" x="80.01" y="125.5014" size="1.778" layer="95" rot="R180"/>
+<attribute name="VALUE" x="80.01" y="130.302" size="1.778" layer="96" rot="R180"/>
+</instance>
+<instance part="R5" gate="G$1" x="76.2" y="124.46" smashed="yes" rot="R180">
+<attribute name="NAME" x="80.01" y="122.9614" size="1.778" layer="95" rot="R180"/>
+<attribute name="VALUE" x="80.01" y="127.762" size="1.778" layer="96" rot="R180"/>
+</instance>
+<instance part="R6" gate="G$1" x="81.28" y="81.28" smashed="yes" rot="R180">
+<attribute name="NAME" x="85.09" y="79.7814" size="1.778" layer="95" rot="R180"/>
+<attribute name="VALUE" x="85.09" y="84.582" size="1.778" layer="96" rot="R180"/>
+</instance>
+<instance part="R7" gate="G$1" x="81.28" y="78.74" smashed="yes" rot="R180">
+<attribute name="NAME" x="85.09" y="77.2414" size="1.778" layer="95" rot="R180"/>
+<attribute name="VALUE" x="85.09" y="82.042" size="1.778" layer="96" rot="R180"/>
+</instance>
+<instance part="R8" gate="G$1" x="81.28" y="20.32" smashed="yes" rot="R180">
+<attribute name="NAME" x="85.09" y="18.8214" size="1.778" layer="95" rot="R180"/>
+<attribute name="VALUE" x="85.09" y="23.622" size="1.778" layer="96" rot="R180"/>
+</instance>
+<instance part="R9" gate="G$1" x="81.28" y="17.78" smashed="yes" rot="R180">
+<attribute name="NAME" x="85.09" y="16.2814" size="1.778" layer="95" rot="R180"/>
+<attribute name="VALUE" x="85.09" y="21.082" size="1.778" layer="96" rot="R180"/>
 </instance>
 </instances>
@@
 <wire x1="111.76" y1="111.76" x2="83.82" y2="111.76" width="0.1524" layer="91"/>
 <wire x1="83.82" y1="111.76" x2="83.82" y2="127" width="0.1524" layer="91"/>
-<pinref part="U3" gate="A" pin="Y"/>
-<wire x1="83.82" y1="127" x2="53.34" y2="127" width="0.1524" layer="91"/>
+<wire x1="83.82" y1="127" x2="81.28" y2="127" width="0.1524" layer="91"/>
+<pinref part="R3" gate="G$1" pin="1"/>
 </segment>
 </net>
@@
 <pinref part="J1" gate="G$1" pin="8"/>
 <wire x1="111.76" y1="109.22" x2="81.28" y2="109.22" width="0.1524" layer="91"/>
-<pinref part="U3" gate="A" pin="Z"/>
 <wire x1="81.28" y1="109.22" x2="81.28" y2="124.46" width="0.1524" layer="91"/>
-<wire x1="81.28" y1="124.46" x2="53.34" y2="124.46" width="0.1524" layer="91"/>
+<pinref part="R5" gate="G$1" pin="1"/>
 </segment>
 </net>
@@
 <wire x1="111.76" y1="68.58" x2="91.44" y2="68.58" width="0.1524" layer="91"/>
 <wire x1="91.44" y1="68.58" x2="91.44" y2="81.28" width="0.1524" layer="91"/>
-<wire x1="91.44" y1="81.28" x2="58.42" y2="81.28" width="0.1524" layer="91"/>
-<wire x1="58.42" y1="81.28" x2="58.42" y2="73.66" width="0.1524" layer="91"/>
-<pinref part="U1" gate="A" pin="Y"/>
-<wire x1="58.42" y1="73.66" x2="53.34" y2="73.66" width="0.1524" layer="91"/>
+<wire x1="91.44" y1="81.28" x2="86.36" y2="81.28" width="0.1524" layer="91"/>
+<pinref part="R6" gate="G$1" pin="1"/>
 </segment>
 </net>
@@
 <wire x1="111.76" y1="60.96" x2="88.9" y2="60.96" width="0.1524" layer="91"/>
 <wire x1="88.9" y1="60.96" x2="88.9" y2="78.74" width="0.1524" layer="91"/>
-<wire x1="88.9" y1="78.74" x2="60.96" y2="78.74" width="0.1524" layer="91"/>
-<wire x1="60.96" y1="78.74" x2="60.96" y2="71.12" width="0.1524" layer="91"/>
-<pinref part="U1" gate="A" pin="Z"/>
-<wire x1="60.96" y1="71.12" x2="53.34" y2="71.12" width="0.1524" layer="91"/>
+<wire x1="88.9" y1="78.74" x2="86.36" y2="78.74" width="0.1524" layer="91"/>
+<pinref part="R7" gate="G$1" pin="1"/>
 </segment>
 </net>
@@
 <wire x1="111.76" y1="58.42" x2="104.14" y2="58.42" width="0.1524" layer="91"/>
 <wire x1="104.14" y1="58.42" x2="104.14" y2="20.32" width="0.1524" layer="91"/>
-<pinref part="U2" gate="A" pin="Y"/>
-<wire x1="104.14" y1="20.32" x2="53.34" y2="20.32" width="0.1524" layer="91"/>
+<wire x1="104.14" y1="20.32" x2="86.36" y2="20.32" width="0.1524" layer="91"/>
+<pinref part="R8" gate="G$1" pin="1"/>
 </segment>
 </net>
@@
 <wire x1="111.76" y1="55.88" x2="106.68" y2="55.88" width="0.1524" layer="91"/>
 <wire x1="106.68" y1="55.88" x2="106.68" y2="17.78" width="0.1524" layer="91"/>
-<pinref part="U2" gate="A" pin="Z"/>
-<wire x1="106.68" y1="17.78" x2="53.34" y2="17.78" width="0.1524" layer="91"/>
+<wire x1="106.68" y1="17.78" x2="86.36" y2="17.78" width="0.1524" layer="91"/>
+<pinref part="R9" gate="G$1" pin="1"/>
 </segment>
 </net>
@@
 </segment>
 </net>
+<net name="N$13" class="0">
+<segment>
+<pinref part="U3" gate="A" pin="Y"/>
+<pinref part="R3" gate="G$1" pin="2"/>
+<wire x1="71.12" y1="127" x2="53.34" y2="127" width="0.1524" layer="91"/>
+</segment>
+</net>
+<net name="N$14" class="0">
+<segment>
+<pinref part="U3" gate="A" pin="Z"/>
+<pinref part="R5" gate="G$1" pin="2"/>
+<wire x1="71.12" y1="124.46" x2="53.34" y2="124.46" width="0.1524" layer="91"/>
+</segment>
+</net>
+<net name="N$15" class="0">
+<segment>
+<pinref part="U1" gate="A" pin="Y"/>
+<pinref part="R6" gate="G$1" pin="2"/>
+<wire x1="76.2" y1="81.28" x2="58.42" y2="81.28" width="0.1524" layer="91"/>
+<wire x1="58.42" y1="81.28" x2="58.42" y2="73.66" width="0.1524" layer="91"/>
+<wire x1="58.42" y1="73.66" x2="53.34" y2="73.66" width="0.1524" layer="91"/>
+</segment>
+</net>
+<net name="N$16" class="0">
+<segment>
+<pinref part="U1" gate="A" pin="Z"/>
+<pinref part="R7" gate="G$1" pin="2"/>
+<wire x1="76.2" y1="78.74" x2="60.96" y2="78.74" width="0.1524" layer="91"/>
+<wire x1="60.96" y1="78.74" x2="60.96" y2="71.12" width="0.1524" layer="91"/>
+<wire x1="60.96" y1="71.12" x2="53.34" y2="71.12" width="0.1524" layer="91"/>
+</segment>
+</net>
+<net name="N$17" class="0">
+<segment>
+<pinref part="U2" gate="A" pin="Y"/>
+<pinref part="R8" gate="G$1" pin="2"/>
+<wire x1="76.2" y1="20.32" x2="53.34" y2="20.32" width="0.1524" layer="91"/>
+</segment>
+</net>
+<net name="N$18" class="0">
+<segment>
+<pinref part="U2" gate="A" pin="Z"/>
+<pinref part="R9" gate="G$1" pin="2"/>
+<wire x1="76.2" y1="17.78" x2="53.34" y2="17.78" width="0.1524" layer="91"/>
+</segment>
+</net>
