File: plug-ins/control/RedPitaya-Support/McBSP-Link-Hardware/MK3-RP-Link/rp-schield-vias.sch (EAGLE design)
At the start: 18 parts, among them U1 SN65MLVD202A, U2 SN65MLVD202A, U3 SN65MLVD202A

Commit message: updated McBSP Link board/schematics updated FPGA bit file for (latest build for V2 Hardware/Interface), design cleanups
Parts:
- added R3, R4, R5: 100R, resistor:R-US_R0402
Connections:
- net CLK+RET-CLKR: now also R5.2
- net CLK-RET-CLKR: now also R5.1
- net CS+-FSX: now also R4.2
- net CS-FSX: now also R4.1
- net MOSI+: now also R3.2
- net MOSI-: now also R3.1
Other:
- note added: "FPGA-S-RX"
- note added: "FPGA-S-TX"

Commit message: updated FPGA init procedure updated -- next gen layout
Parts:
- added R10, R11, R6, R7, R8, R9: 25R, resistor:R-US_R0402
- added R12, R13: 0R, resistor:R-US_M1206
- R1, R2: value 24R9 -> XXR
Connections:
- net FPGA-S-CLK renamed CLKX
- new net N$1: R6.2, U3.Y
- new net N$3: R7.2, U3.Z
- new net N$4: R8.2, U1.Y
- new net N$5: R9.2, U1.Z
- new net N$7: R10.2, U2.Y
- new net N$8: R11.2, U2.Z
- net CLK+-CLKX: now also R10.1; no longer U2.Y
- net CLK--CLKX: now also R11.1; no longer U2.Z
- net CS+RET-FSR: now also R8.1; no longer U1.Y
- net CS-RET-FSR: now also R9.1; no longer U1.Z
- net FSP: now also R13.1
- net MISO+: now also R6.1; no longer U3.Y
- net MISO-: now also R7.1; no longer U3.Z
- net N$10: now also R12.1
- net N$2: now also R12.2
- net N$6: now also R13.2
Other:
- note added: "CLKR-FPGA"
- moved on the sheet: R1, R2
